File: pcb/ergosnap.sch (KiCad schematic (older format))
At the start: 41 parts, among them J0 Conn_01x05_Female, J1 5PIN, SW1 switch_diode, SW10 switch_diode, SW11 switch_diode, SW12 switch_diode, SW13 switch_diode, SW14 switch_diode, SW15 switch_diode, SW16 switch_diode, SW17 switch_diode, SW18 switch_diode, SW19 switch_diode, SW2 switch_diode, SW20 switch_diode, SW21 switch_diode, SW22 switch_diode, SW23 switch_diode, SW24 switch_diode, SW25 switch_diode, SW26 switch_diode, SW27 switch_diode, SW28 switch_diode, SW3 switch_diode, SW30 switch_diode, SW31 switch_diode, SW32 switch_diode, SW33 switch_diode, SW34 switch_diode, SW35 switch_diode, SW4 switch_diode, SW5 switch_diode, SW6 switch_diode, SW7 switch_diode, SW8 switch_diode, SW9 switch_diode, U3 ProMicro

Commit message: Rev1.1 final (?)
- Added reset header
- Reshaped the bottom of the board slightly
- Moved most of the component references off the silkscreen
- Marked pin 1 in ProMicro footprint
- Added 2 switch traces missed in last update
Parts:
- added J2: Conn_01x02_Female, Connector_Wire:SolderWirePad_1x02_P3.81mm_Drill0.8mm, symbol Connector:Conn_01x02_Female
Connections:
- net labels added: rst
- wire segments 236 -> 239
Changed lines of the file:
@@
 	0    -1   -1   0
 $EndComp
+$Comp
+L Connector:Conn_01x02_Female J2
+U 1 1 5D3D1108
+P 2400 2600
+F 0 "J2" H 2428 2576 50  0000 L CNN
+F 1 "Conn_01x02_Female" H 2428 2485 50  0000 L CNN
+F 2 "Connector_Wire:SolderWirePad_1x02_P3.81mm_Drill0.8mm" H 2400 2600 50  0001 C CNN
+F 3 "~" H 2400 2600 50  0001 C CNN
+	1    2400 2600
+	1    0    0    -1
+$EndComp
+Wire Wire Line
+	2200 2600 2050 2600
+Wire Wire Line
+	2200 2700 2050 2700
+Text Label 2050 2600 0    50   ~ 0
+rst
+Text Label 2050 2700 0    50   ~ 0
+GND
+Wire Wire Line
+	2700 3350 3000 3350
+Text Label 3000 3350 0    50   ~ 0
+rst
 $EndSCHEMATC
